Commit message: Tuned values for mass, damping etc

File: autocar_description/urdf/autocar.xacro (robot description, xacro)
@@ -27,5 +27,5 @@
 limitations under the License.
 -->
-<robot name="em_3905" xmlns:xacro="http://www.ros.org/wiki/xacro">
+<robot name="autocar" xmlns:xacro="http://www.ros.org/wiki/xacro">
   <xacro:include filename="$(find autocar_description)/urdf/autocar.gazebo"/>
   <!-- Degree-to-radian conversions -->
@@ -34,20 +34,8 @@
   <!-- chassis_length is measured along the x axis, chassis_width
        along the y axis, and chassis_height along the z axis. -->
-  <xacro:property name="chassis_length" value="0.20837"/>
-  <xacro:property name="chassis_width" value="0.1010"/>
-  <xacro:property name="chassis_height" value="0.046"/>
-  <xacro:property name="chassis_mass" value="1.0019"/>
-  <!-- battery_dist is the distance between the inner edges of the
-       batteries. battery_comp_depth is the battery compartment depth.
-       battery_length is measured along the x axis, battery_width
-       along the y axis, and battery_height along the z axis. -->
-  <xacro:property name="battery_x_offset" value="0.055"/>
-  <xacro:property name="battery_dist" value="0.065"/>
-  <xacro:property name="battery_comp_depth" value="0.02"/>
-  <xacro:property name="battery_comp_angle" value="0.34906585"/>
-  <xacro:property name="battery_length" value="0.16"/>
-  <xacro:property name="battery_width" value="0.047"/>
-  <xacro:property name="battery_height" value="0.024"/>
-  <xacro:property name="battery_mass" value="0.5025"/>
+  <xacro:property name="chassis_length" value="0.2141"/>
+  <xacro:property name="chassis_width" value="0.139"/>
+  <xacro:property name="chassis_height" value="0.01"/>
+  <xacro:property name="chassis_mass" value="1.009"/>
   <!-- hub_dia and tire_dia are the diameters of the hub and tire,
        respectively. hex_hub_depth is the distance that the hex hub is
@@ -55,18 +43,18 @@
        is a "zero offset" wheel. hex_hub_depth = tire_width / 2 -
        axle_length. -->
-  <xacro:property name="hub_dia" value="0.09652"/>
-  <xacro:property name="tire_dia" value="0.14605"/>
-  <xacro:property name="tire_width" value="0.0889"/>
-  <xacro:property name="hex_hub_depth" value="0.01445"/>
-  <xacro:property name="wheel_mass" value="0.29"/>
+  <xacro:property name="hub_dia" value="0.0801"/>
+  <xacro:property name="tire_dia" value="0.1212"/>
+  <xacro:property name="tire_width" value="0.0737"/>
+  <xacro:property name="hex_hub_depth" value="0.01195"/>
+  <xacro:property name="wheel_mass" value="0.2407"/>
   <!-- hex_hub_dist is the distance between left and right hex hubs when
        the shock absorbers are fully extended. axle_length is the distance
        from a U joint to the corresponding hex hub. wheel_travel is the
        vertical wheel travel. -->
-  <xacro:property name="wheelbase" value="0.335"/>
-  <xacro:property name="hex_hub_dist" value="0.365"/>
-  <xacro:property name="axle_length" value="0.03"/>
-  <xacro:property name="wheel_travel" value="0.084"/>
-  <xacro:property name="shock_z_offset" value="0.120"/>
+  <xacro:property name="wheelbase" value="0.27805"/>
+  <xacro:property name="hex_hub_dist" value="0.30295"/>
+  <xacro:property name="axle_length" value="0.0243"/>
+  <xacro:property name="wheel_travel" value="0.06972"/>
+  <xacro:property name="shock_z_offset" value="0.09"/>
   <!-- shock_eff_limit is 2 * ((shock_stroke / 2) * shock_spring_constant) N.
        shock_stroke is 0.028575 meters. shock_spring_constant, an approximation
@@ -155,5 +143,5 @@
     <gazebo reference="${lr_prefix}_${fr_prefix}_shock">
         <implicitSpringDamper>true</implicitSpringDamper>
-        <springStiffness>91.13</springStiffness>
+        <springStiffness>91.37</springStiffness>
         <springReference>0.028575</springReference>
     </gazebo>
@@ -172,5 +160,5 @@
       <axis xyz="0 0 -1"/>
       <limit effort="${axle_eff_limit}" velocity="${axle_vel_limit}"/>
-      <dynamics damping="1E-4" friction="1E-5"/>
+      <dynamics damping="1E-4" friction="1E-6"/>
     </joint>
     <link name="${lr_prefix}_${fr_prefix}_wheel">
@@ -217,5 +205,5 @@
       <limit lower="${-degrees_45}" upper="${degrees_45}"
              effort="${servo_stall_torque}" velocity="${servo_no_load_speed}"/>
-      <dynamics damping="1E-4" friction="1E-5"/>
+      <dynamics damping="1E-4" friction="0.1"/>
     </joint>
     <xacro:wheel lr_prefix="${lr_prefix}" fr_prefix="${fr_prefix}"

Commit message: Added dynamic reconfigure for PID parameters

File: autocar_description/urdf/autocar.xacro (robot description, xacro)
@@ -205,5 +205,5 @@
       <limit lower="${-degrees_45}" upper="${degrees_45}"
              effort="${servo_stall_torque}" velocity="${servo_no_load_speed}"/>
-      <dynamics damping="1E-4" friction="0.1"/>
+      <dynamics damping="0.0089" friction="0.1"/>
     </joint>
     <xacro:wheel lr_prefix="${lr_prefix}" fr_prefix="${fr_prefix}"

Commit message: Tuned some values for damping and frction for wheels Tuned PID parameters

File: autocar_description/urdf/autocar.xacro (robot description, xacro)
@@ -47,5 +47,5 @@
   <xacro:property name="tire_width" value="0.0737"/>
   <xacro:property name="hex_hub_depth" value="0.01195"/>
-  <xacro:property name="wheel_mass" value="0.2407"/>
+  <xacro:property name="wheel_mass" value="0.098"/>
   <!-- hex_hub_dist is the distance between left and right hex hubs when
        the shock absorbers are fully extended. axle_length is the distance
@@ -56,5 +56,5 @@
   <xacro:property name="axle_length" value="0.0243"/>
   <xacro:property name="wheel_travel" value="0.06972"/>
-  <xacro:property name="shock_z_offset" value="0.09"/>
+  <xacro:property name="shock_z_offset" value="0.065"/>
   <!-- shock_eff_limit is 2 * ((shock_stroke / 2) * shock_spring_constant) N.
        shock_stroke is 0.028575 meters. shock_spring_constant, an approximation
@@ -80,5 +80,5 @@
        6 V. servo_stall_torque is measured in N m. servo_no_load_speed is
        measured in rad/s. -->
-  <xacro:property name="servo_stall_torque" value="0.5649"/>
+  <xacro:property name="servo_stall_torque" value="2.4"/>
   <xacro:property name="servo_no_load_speed" value="4.553"/>
   <material name="chassis_mat">
@@ -139,10 +139,10 @@
       <limit lower="${-wheel_travel / 2}" upper="${wheel_travel / 2}"
              effort="${shock_eff_limit}" velocity="${shock_vel_limit}"/>
-      <dynamics damping="3.8"/>
+      <dynamics damping="38" friction="0.75"/>
     </joint>
     <gazebo reference="${lr_prefix}_${fr_prefix}_shock">
         <implicitSpringDamper>true</implicitSpringDamper>
-        <springStiffness>91.37</springStiffness>
-        <springReference>0.028575</springReference>
+        <springStiffness>91.75</springStiffness>
+        <springReference>0.028375</springReference>
     </gazebo>
   </xacro:macro>
@@ -160,5 +160,5 @@
       <axis xyz="0 0 -1"/>
       <limit effort="${axle_eff_limit}" velocity="${axle_vel_limit}"/>
-      <dynamics damping="1E-4" friction="1E-6"/>
+      <dynamics damping="0.001" friction="0.01"/>
     </joint>
     <link name="${lr_prefix}_${fr_prefix}_wheel">
@@ -205,5 +205,5 @@
       <limit lower="${-degrees_45}" upper="${degrees_45}"
              effort="${servo_stall_torque}" velocity="${servo_no_load_speed}"/>
-      <dynamics damping="0.0089" friction="0.1"/>
+      <dynamics damping="1E-4" friction="0.1"/>
     </joint>
     <xacro:wheel lr_prefix="${lr_prefix}" fr_prefix="${fr_prefix}"

Commit message: Added tele operation using key and dual-shock controller. Removed driving joints when the Ackermann message is not received in plugin.

File: autocar_description/urdf/autocar.xacro (robot description, xacro)
@@ -160,5 +160,5 @@
       <axis xyz="0 0 -1"/>
       <limit effort="${axle_eff_limit}" velocity="${axle_vel_limit}"/>
-      <dynamics damping="0.001" friction="0.01"/>
+      <dynamics damping="0.0001" friction="0.01"/>
     </joint>
     <link name="${lr_prefix}_${fr_prefix}_wheel">

Commit message: Added IMU sensor and added launch file to launch rviz and robot_state_publisher

File: autocar_description/urdf/autocar.xacro (robot description, xacro)
@@ -38,4 +38,9 @@
   <xacro:property name="chassis_height" value="0.01"/>
   <xacro:property name="chassis_mass" value="1.009"/>
+  <!-- Rough measurements for Waveshare Sense hat -->
+  <xacro:property name="imu_sensor_length" value="0.030"/>
+  <xacro:property name="imu_sensor_width" value="0.065"/>
+  <xacro:property name="imu_sensor_height" value="0.008"/>
+  <xacro:property name="imu_sensor_z_position" value="0.02"/>
   <!-- hub_dia and tire_dia are the diameters of the hub and tire,
        respectively. hex_hub_depth is the distance that the hex hub is
@@ -256,8 +261,49 @@
     <material>Gazebo/Grey</material>
   </gazebo>
+  <!-- IMU link -->
+  <link name="imu_link">
+    <xacro:null_inertial/>
+    <visual name="imu_visual">
+      <origin xyz="-${chassis_length/4} 0.0 ${imu_sensor_z_position}" rpy="0.0 0.0 0.0"/>
+      <geometry>
+        <box size="${imu_sensor_length} ${imu_sensor_width} ${imu_sensor_height}"/>
+      </geometry>
+      <material name="imu_mat">
+        <color rgba="1.0 0.0 0.0 1.0"/>
+      </material>
+    </visual>
+  </link>
+  <gazebo reference="imu_link">
+    <material>Gazebo/Red</material>
+  </gazebo>
   <joint name="base_link_to_chasis" type="fixed">
     <parent link="base_link"/>
     <child link="chassis"/>
   </joint>
+  <joint name="imu_to_chassis" type="fixed">
+    <parent link="chassis"/>
+    <child link="imu_link"/>
+  </joint>
+  <!-- IMU Plugin -->
+    <gazebo reference="imu_link">
+    <gravity>true</gravity>
+    <sensor name="imu_sensor" type="imu">
+      <always_on>true</always_on>
+      <update_rate>220</update_rate>
+      <visualize>true</visualize>
+      <topic>__default_topic__</topic>
+      <plugin filename="libgazebo_ros_imu_sensor.so" name="imu_plugin">
+        <topicName>imu</topicName>
+        <bodyName>imu_link</bodyName>
+        <updateRateHZ>220.0</updateRateHZ>
+        <gaussianNoise>0.0</gaussianNoise>
+        <xyzOffset>0 0 0</xyzOffset>
+        <rpyOffset>0 0 0</rpyOffset>
+        <frameName>imu_link</frameName>
+        <initialOrientationAsReference>false</initialOrientationAsReference>
+      </plugin>
+      <pose>0 0 0 0 0 0</pose>
+    </sensor>
+  </gazebo>
   <!-- Wheels -->
   <xacro:front_wheel lr_prefix="left" fr_prefix="front"

Commit message: Added rplidar to the car

File: autocar_description/urdf/autocar.xacro (robot description, xacro)
@@ -277,14 +277,40 @@
     <material>Gazebo/Red</material>
   </gazebo>
+  <!-- Lidar link -->
+  <link name="rp_lidar">
+    <collision>
+      <origin xyz="${chassis_length/4} 0.0 ${imu_sensor_z_position}" rpy="1.5707 0 4.71"/>
+      <geometry>
+        <mesh filename="package://autocar_description/meshes/rplidar.dae" scale="0.001 0.001 0.001" />
+      </geometry>
+    </collision>
+    <visual>
+      <origin xyz="${chassis_length/4} 0.0 ${imu_sensor_z_position}" rpy="1.5707 0 4.71"/>
+      <geometry>
+        <mesh filename="package://autocar_description/meshes/rplidar.dae" scale="0.001 0.001 0.001" />
+      </geometry>
+    </visual>
+    <inertial>
+      <mass value="1e-5" />
+      <origin xyz="${chassis_length/4} 0.0 ${imu_sensor_z_position}" rpy="1.5707 0 4.71"/>
+      <inertia ixx="0" ixy="0" ixz="0" iyy="0" iyz="0" izz="0" />
+    </inertial>
+  </link>
   <joint name="base_link_to_chasis" type="fixed">
     <parent link="base_link"/>
     <child link="chassis"/>
   </joint>
+  <!-- IMU joint -->
   <joint name="imu_to_chassis" type="fixed">
     <parent link="chassis"/>
     <child link="imu_link"/>
   </joint>
+  <!-- Lidar joint -->
+  <joint name="rplidar_joint" type="fixed">
+    <parent link="base_link"/>
+    <child link="rp_lidar"/>
+  </joint>
   <!-- IMU Plugin -->
-    <gazebo reference="imu_link">
+  <gazebo reference="imu_link">
     <gravity>true</gravity>
     <sensor name="imu_sensor" type="imu">

Commit message: Added rplidar to the car
# Conflicts:
#	autocar_description/urdf/autocar.gazebo
#	autocar_description/urdf/autocar.xacro

File: autocar_description/urdf/autocar.xacro (robot description, xacro)
@@ -277,11 +277,37 @@
     <material>Gazebo/Red</material>
   </gazebo>
+  <!-- Lidar link -->
+  <link name="rp_lidar">
+    <collision>
+      <origin xyz="${chassis_length/4} 0.0 ${imu_sensor_z_position}" rpy="1.5707 0 4.71"/>
+      <geometry>
+        <mesh filename="package://autocar_description/meshes/rplidar.dae" scale="0.001 0.001 0.001" />
+      </geometry>
+    </collision>
+    <visual>
+      <origin xyz="${chassis_length/4} 0.0 ${imu_sensor_z_position}" rpy="1.5707 0 4.71"/>
+      <geometry>
+        <mesh filename="package://autocar_description/meshes/rplidar.dae" scale="0.001 0.001 0.001" />
+      </geometry>
+    </visual>
+    <inertial>
+      <mass value="1e-5" />
+      <origin xyz="${chassis_length/4} 0.0 ${imu_sensor_z_position}" rpy="1.5707 0 4.71"/>
+      <inertia ixx="0" ixy="0" ixz="0" iyy="0" iyz="0" izz="0" />
+    </inertial>
+  </link>
   <joint name="base_link_to_chasis" type="fixed">
     <parent link="base_link"/>
     <child link="chassis"/>
   </joint>
+  <!-- IMU joint -->
   <joint name="imu_to_chassis" type="fixed">
     <parent link="chassis"/>
     <child link="imu_link"/>
+  </joint>
+  <!-- Lidar joint -->
+  <joint name="rplidar_joint" type="fixed">
+    <parent link="base_link"/>
+    <child link="rp_lidar"/>
   </joint>
   <!-- Wheels -->

Commit message: Added lidar and fixed problems with it.

File: autocar_description/urdf/autocar.xacro (robot description, xacro)
@@ -43,4 +43,6 @@
   <xacro:property name="imu_sensor_height" value="0.008"/>
   <xacro:property name="imu_sensor_z_position" value="0.02"/>
+  <!-- Rough estimates for the Lidar position -->
+  <xacro:property name="lidar_z_position" value="0.04"/>
   <!-- hub_dia and tire_dia are the diameters of the hub and tire,
        respectively. hex_hub_depth is the distance that the hex hub is
@@ -280,5 +282,5 @@
   <link name="rp_lidar">
     <collision>
-      <origin xyz="${chassis_length/4} 0.0 ${imu_sensor_z_position}" rpy="1.5707 0 4.71"/>
+      <origin xyz="${chassis_length/4} 0.0 0.0" rpy="1.5707 0 4.71"/>
       <geometry>
         <mesh filename="package://autocar_description/meshes/rplidar.dae" scale="0.001 0.001 0.001" />
@@ -286,5 +288,5 @@
     </collision>
     <visual>
-      <origin xyz="${chassis_length/4} 0.0 ${imu_sensor_z_position}" rpy="1.5707 0 4.71"/>
+      <origin xyz="${chassis_length/4} 0.0 0.0" rpy="1.5707 0 4.71"/>
       <geometry>
         <mesh filename="package://autocar_description/meshes/rplidar.dae" scale="0.001 0.001 0.001" />
@@ -293,5 +295,5 @@
     <inertial>
       <mass value="1e-5" />
-      <origin xyz="${chassis_length/4} 0.0 ${imu_sensor_z_position}" rpy="1.5707 0 4.71"/>
+      <origin xyz="${chassis_length/4} 0.0 0.0" rpy="1.5707 0 4.71"/>
       <inertia ixx="0" ixy="0" ixz="0" iyy="0" iyz="0" izz="0" />
     </inertial>
@@ -308,6 +310,7 @@
   <!-- Lidar joint -->
   <joint name="rplidar_joint" type="fixed">
-    <parent link="base_link"/>
+    <parent link="chassis"/>
     <child link="rp_lidar"/>
+    <origin xyz="0.0 0 ${lidar_z_position}" rpy="0 0 0"/>
   </joint>
   <!-- Wheels -->
